File: Type 1 Termination Board v3.sch (KiCad schematic (older format))
At the start: 3 parts, among them J2 Conn_01x01_Female, J3 Conn_01x01_Female, J4 Conn_01x05

Commit message: Add files via upload
Connections:
- net LV: now reaches J2.1 (Pin_1), J4.1 (Pin_1), J4.2 (Pin_2)
- net return: now reaches J3.1 (Pin_1), J4.4 (Pin_4), J4.5 (Pin_5)
Changed lines of the file:
@@
 EESchema Schematic File Version 4
+LIBS:Type 1 Termination Board v3-cache
 EELAYER 29 0
 EELAYER END
@@
 Text HLabel 1660 2770 1    50   Input ~ 0
 GND
+Text HLabel 1840 2600 1    50   Input ~ 0
+LV
+Text HLabel 1990 2960 3    50   Input ~ 0
+return
 $EndSCHEMATC
