File: Type 1 Termination Board v3.kicad_pcb (KiCad board)
At the start: 4 copper layers, 53 x 20.3 mm, 13 parts, among them J2 Conn_01x01_Female, J3 Conn_01x01_Female

Commit message: Add files via upload
Parts:
- J10: renamed from UMPS; value Conn_01x05 -> UMPS
- J11: renamed from TLH; value 19-1_TLH_HV -> TLH
- J12: renamed from TLH; value 20 Pin -> TLH
Routing:
- net /return: vias 25 -> 18
Other:
- board text added: "Quad1"
- board text added: "Quad2"
- board text added: "Quad3"
- board text added: "Quad4"
- board text added: "Quad_rtn"
- board text added: "Trip1"
- board text added: "Trip2"
- board text added: "Trip3"
- board text added: "Trip4"
- board text added: "Trip_rtn"

Commit message: Add files via upload
Parts:
- renumbered REF** to J20, REF** to J21, REF** to J22, REF** to J23, REF** to P1, REF** to P2, REF** to P3, REF** to P4
Other:
- board text added: "+Cp1"
- board text added: "+Cp2"
- board text added: "+Tint1"
- board text added: "+Vc1"
- board text added: "+Vc2"
- board text added: "-"
- board text added: "P1r"
- board text added: "P2r"
- board text added: "Q1"
- board text added: "Q2"
- board text added: "Q3"
- board text added: "Q4"
- board text added: "Q_rtn"
- board text added: "T1"
- board text added: "T2"
- board text added: "T3"
- board text added: "T4"
- board text added: "T_rtn"
- board text removed: "Add ground pads for LP1 and LP2"
- board text removed: "Cp1+"
- board text removed: "Cp1-"
- board text removed: "Cp2+"
- board text removed: "Cp2-"
- board text removed: "IntT1+"
- board text removed: "IntT1-"
- board text removed: "IntT2+"
- board text removed: "IntT2-"
- board text removed: "IntT3+"
- board text removed: "IntT3-"
- board text removed: "LP1_rtn"
- board text removed: "LP2_rtn"
- board text removed: "Quad1"
- board text removed: "Quad2"
- board text removed: "Quad3"
- board text removed: "Quad4"
- board text removed: "Quad_rtn"
- board text removed: "Trip1"
- board text removed: "Trip2"
- board text removed: "Trip3"
- board text removed: "Trip4"
- board text removed: "Trip_rtn"
- board text removed: "Vc1+"
- board text removed: "Vc1-"
- board text removed: "Vc2+"
- board text removed: "Vc2-"
